File: moc/MCU board/mcu_board/mcu_board.kicad_pcb (KiCad board)
At the start: 2 copper layers, 41 x 30 mm, 10 parts, among them J1 Conn_01x04_Female, J2 Conn_01x05_Female, J3 Conn_01x05_Male, J4 Conn_01x09_Female, J5 Conn_01x09_Female, U1 ATtiny861V-10SU

Commit message: Plots ready
Routing:
- net PB1: track 15.1 -> 18.1 mm
- net GND: vias 1 -> 3
- added copper zone on F.Cu, net (none)
Changed lines of the file:
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@@
   (general
     (thickness 1.6)
-    (drawings 4)
-    (tracks 151)
+    (drawings 8)
+    (tracks 154)
     (zones 0)
     (modules 10)
@@
     (via_min_size 0.4)
     (via_min_drill 0.3)
-    (user_via 1.65 0.8)
+    (user_via 1.65 0.6)
     (uvia_size 0.3)
     (uvia_drill 0.1)
@@
     (visible_elements 7FFFFFFF)
     (pcbplotparams
-      (layerselection 0x010fc_ffffffff)
+      (layerselection 0x01000_ffffffff)
       (usegerberextensions false)
       (usegerberattributes true)
@@
       (excludeedgelayer true)
       (linewidth 0.100000)
-      (plotframeref false)
+      (plotframeref true)
       (viasonmask false)
       (mode 1)
@@
       (psnegative false)
       (psa4output false)
-      (plotreference true)
-      (plotvalue true)
+      (plotreference false)
+      (plotvalue false)
       (plotinvisibletext false)
       (padsonsilk false)
       (subtractmaskfromsilk false)
-      (outputformat 1)
-      (mirror false)
+      (outputformat 5)
+      (mirror true)
       (drillshape 1)
       (scaleselection 1)
-      (outputdirectory ""))
+      (outputdirectory "./"))
   )
   (net 0 "")
@@
     (add_net MOSI)
     (add_net "Net-(C3-Pad2)")
-    (add_net "Net-(U1-Pad7)")
-    (add_net "Net-(U1-Pad8)")
     (add_net PB1)
     (add_net PB2)
@@
       (effects (font (size 0.8 0.8) (thickness 0.12)) (justify mirror))
     )
-    (pad 1 smd roundrect (at -1.6625 0 180) (size 1.225 1.9) (layers B.Cu B.Paste B.Mask) (roundrect_rratio 0.204082)
+    (pad 1 smd roundrect (at -1.6625 0 180) (size 1.225 1.9) (layers B.Cu B.Paste B.Mask) (roundrect_rratio 0.2040816326530612)
       (net 2 VCC))
-    (pad 2 smd roundrect (at 1.6625 0 180) (size 1.225 1.9) (layers B.Cu B.Paste B.Mask) (roundrect_rratio 0.204082)
+    (pad 2 smd roundrect (at 1.6625 0 180) (size 1.225 1.9) (layers B.Cu B.Paste B.Mask) (roundrect_rratio 0.2040816326530612)
       (net 3 "Net-(C3-Pad2)"))
     (model ${KISYS3DMOD}/Inductor_SMD.3dshapes/L_1206_3216Metric.wrl
@@
       (effects (font (size 0.8 0.8) (thickness 0.12)) (justify mirror))
     )
-    (pad 1 smd roundrect (at -1.5625 0 270) (size 1.325 1.8) (layers B.Cu B.Paste B.Mask) (roundrect_rratio 0.188679)
-      (net 1 GND))
-    (pad 2 smd roundrect (at 1.5625 0 270) (size 1.325 1.8) (layers B.Cu B.Paste B.Mask) (roundrect_rratio 0.188679)
+    (pad 1 smd roundrect (at -1.5625 0 270) (size 1.325 1.8) (layers B.Cu B.Paste B.Mask) (roundrect_rratio 0.1886784905660377)
+      (net 1 GND))
+    (pad 2 smd roundrect (at 1.5625 0 270) (size 1.325 1.8) (layers B.Cu B.Paste B.Mask) (roundrect_rratio 0.1886784905660377)
       (net 2 VCC))
     (model ${KISYS3DMOD}/Capacitor_SMD.3dshapes/C_1206_3216Metric.wrl
@@
       (effects (font (size 0.8 0.8) (thickness 0.12)) (justify mirror))
     )
-    (pad 2 smd roundrect (at 1.5625 0 90) (size 1.325 1.8) (layers B.Cu B.Paste B.Mask) (roundrect_rratio 0.188679)
+    (pad 2 smd roundrect (at 1.5625 0 90) (size 1.325 1.8) (layers B.Cu B.Paste B.Mask) (roundrect_rratio 0.1886784905660377)
       (net 3 "Net-(C3-Pad2)"))
-    (pad 1 smd roundrect (at -1.5625 0 90) (size 1.325 1.8) (layers B.Cu B.Paste B.Mask) (roundrect_rratio 0.188679)
+    (pad 1 smd roundrect (at -1.5625 0 90) (size 1.325 1.8) (layers B.Cu B.Paste B.Mask) (roundrect_rratio 0.1886784905660377)
       (net 1 GND))
     (model ${KISYS3DMOD}/Capacitor_SMD.3dshapes/C_1206_3216Metric.wrl
@@
     )
   )
+  (target plus (at 73 64) (size 5) (width 0.05) (layer Edge.Cuts))
+  (target plus (at 120 64) (size 5) (width 0.05) (layer Edge.Cuts))
+  (target plus (at 120 100) (size 5) (width 0.05) (layer Edge.Cuts))
+  (target plus (at 73 100) (size 5) (width 0.05) (layer Edge.Cuts))
   (gr_line (start 117 97) (end 117 67) (layer Edge.Cuts) (width 0.05))
   (gr_line (start 76 97) (end 76 67) (layer Edge.Cuts) (width 0.05))
@@
   (segment (start 100 69) (end 100 72) (width 0.6) (layer B.Cu) (net 1))
   (segment (start 100 72) (end 99.54051 72) (width 0.6) (layer B.Cu) (net 1))
-  (via (at 95 74) (size 1.65) (drill 0.8) (layers F.Cu B.Cu) (net 1))
+  (via (at 94 74) (size 1.65) (drill 0.8) (layers F.Cu B.Cu) (net 1))
+  (via (at 90 88) (size 1.65) (drill 0.8) (layers F.Cu B.Cu) (net 1))
+  (via (at 85 83) (size 1.65) (drill 0.8) (layers F.Cu B.Cu) (net 1))
   (segment (start 88.0725 80.635) (end 89.35 80.635) (width 0.6) (layer B.Cu) (net 2))
   (segment (start 85 77.5625) (end 88.0725 80.635) (width 0.6) (layer B.Cu) (net 2))
@@
   (segment (start 97 73.62) (end 92.38 69) (width 0.381) (layer B.Cu) (net 14))
   (segment (start 97 74.93) (end 97 73.62) (width 0.381) (layer B.Cu) (net 14))
-  (segment (start 92.53 73) (end 91.3 73) (width 0.381) (layer B.Cu) (net 15))
   (segment (start 91.3 73) (end 87.3 69) (width 0.381) (layer B.Cu) (net 15))
-  (segment (start 97.625 78.095) (end 92.53 73) (width 0.381) (layer B.Cu) (net 15))
   (segment (start 98.65 78.095) (end 97.625 78.095) (width 0.381) (layer B.Cu) (net 15))
+  (segment (start 91.3 73) (end 91.3 76.3) (width 0.381) (layer B.Cu) (net 15))
+  (segment (start 93.095 78.095) (end 98.65 78.095) (width 0.381) (layer B.Cu) (net 15))
+  (segment (start 91.3 76.3) (end 93.095 78.095) (width 0.381) (layer B.Cu) (net 15))
   (via (at 102 76) (size 1.65) (drill 0.8) (layers F.Cu B.Cu) (net 16))
   (segment (start 101.175 76.825) (end 102 76) (width 0.381) (layer B.Cu) (net 16))
@@
     (polygon
       (pts
+        (xy 117 97) (xy 76 97) (xy 76 67) (xy 117 67)
+      )
+    )
+  )
+  (zone (net 0) (net_name "") (layer F.Cu) (hatch edge 0.508)
+    (connect_pads (clearance 0.508))
+    (min_thickness 0.254)
+    (fill yes (arc_segments 32) (thermal_gap 0.508) (thermal_bridge_width 0.508))
+    (polygon
+      (pts
+        (xy 117 97) (xy 76 97) (xy 76 67) (xy 117 67)
+      )
+    )
+  )
+  (zone (net 1) (net_name GND) (layer B.Cu) (hatch edge 0.508)
+    (connect_pads yes (clearance 0.508))
+    (min_thickness 0.254)
+    (fill yes (arc_segments 32) (thermal_gap 0.508) (thermal_bridge_width 0.508) (smoothing chamfer))
+    (polygon
+      (pts

Commit message: first protoype
Parts:
- C1: footprint Capacitor_THT:CP_Radial_Tantal_D5.0mm_P2.50mm -> Capacitor_THT:CP_Radial_D4.0mm_P1.50mm; moved to F.Cu
- J1: value Conn_01x04_Female -> Conn_02x03_Counter_Clockwise; footprint Connector_PinSocket_2.54mm:PinSocket_1x04_P2.54mm_Vertical -> .Ambisonic:ICSP_Header_P2.54_SelfSolder; moved to F.Cu
- J2, J3: moved to F.Cu
- J4, J5: footprint Connector_PinSocket_2.54mm:PinSocket_1x09_P2.54mm_Vertical -> .Ambisonic:Header-01x09-p2.54-selfsolder; moved to B.Cu
- moved J4 40.1 mm to (106.9, 122.5), turned to 0 degrees
- moved J1 40.1 mm to (101.2, 115.0), turned to 90 degrees
- moved C1 37.3 mm to (96.5, 108.5), turned to 0 degrees
- moved U1 35.6 mm to (113.2, 110.0)
- moved L1 31.9 mm to (128.0, 103.0), turned to -90 degrees
- moved C2 31.5 mm to (98.5, 104.5), turned to 180 degrees
- moved C3 30.4 mm to (123.0, 103.0), turned to -90 degrees
- moved J2 30.0 mm to (122.9, 115.1)
- moved J5 29.8 mm to (107.0, 98.0), turned to 180 degrees
- moved J3 27.1 mm to (123.0, 97.0)
Connections:
- net PB1 renamed BUT1
- net PB2 renamed BUT2
- net PB3 renamed BUT3
- C1 pad 1: GND -> VCC
- C1 pad 2: VCC -> GND
- J1 pad 1: PSFHCLK -> MISO
- J1 pad 2: ENCB -> PSFHCLK
- J1 pad 3: MISO -> ENCB
- J1 pad 4: MOSI -> VCC
- J4 pad 1: MISO -> BUT0
- J4 pad 3: MOSI -> MISO
- U1 pad 1: MOSI -> BUT0
- U1 pad 7: (no net) -> unconnected-(U1-Pad7)
- U1 pad 8: (no net) -> unconnected-(U1-Pad8)
Routing:
- net BUT0: track 0.00 -> 24.5 mm, vias 0 -> 2
- net MOSI: track 18.4 -> 0.00 mm
- net GND: track 137.0 -> 128.5 mm, vias 3 -> 5
- net PSFHCLK: track 26.3 -> 18.3 mm, vias 0 -> 2
- net SDA: track 32.9 -> 25.4 mm, vias 0 -> 1
- net VCC: track 111.3 -> 105.0 mm, vias 2 -> 5
- net Net-(C3-Pad2): track 7.21 -> 13.3 mm
- net ENCB: track 25.7 -> 20.2 mm
- net MISO: track 18.0 -> 12.6 mm
- net ADC0: track 10.8 -> 13.1 mm
- net ENCSW: track 26.4 -> 24.2 mm, vias 1 -> 2
- net ADC1: track 5.78 -> 7.62 mm
- net SCL: track 30.3 -> 31.7 mm, vias 0 -> 1
- net PSHFUPDATE: track 14.7 -> 15.5 mm
- net BUT1: track 18.1 -> 17.6 mm
- removed copper zone on F.Cu, net (none)
Other:
- board size 41 x 30 mm -> 41.5 x 30 mm
- net class Default removed
- net class VCC removed
