File: moc/Mainboard-pcb/controller_motion_pcb.sch (KiCad schematic (older format))
At the start: 20 parts, among them J1 Conn_01x14_Male, J3 Conn_01x15_Male, P0 Conn_01x03, P1 Conn_01x03, P2 Conn_01x03, P3 Conn_01x03, P4 Conn_01x03, P5 Conn_01x03, P6 Conn_01x03, P7 Conn_01x03

Commit message: first commit
Parts:
- removed BtnMx1: Conn_02x09_Counter_Clockwise, Connector_IDC:IDC-Header_2x10_P2.54mm_Vertical, symbol controller_motion_pcb-rescue:Conn_02x10_Counter_Clockwise-Connector_Generic
- removed CTR1: Teensy4.1, teensy:Teensy41, symbol controller_motion_pcb-rescue:Teensy4.1-teensy
- removed ENC0, ENC1, ENC2, ENC3: Conn_01x05, Connector_JST:JST_EH_B5B-EH-A_1x05_P2.50mm_Vertical, symbol controller_motion_pcb-rescue:Conn_01x05-Connector_Generic
- removed J1: Conn_01x14_Male, Connector_PinHeader_2.54mm:PinHeader_1x14_P2.54mm_Vertical, symbol controller_motion_pcb-rescue:Conn_01x14_Male-Connector
- removed J3: Conn_01x15_Male, Connector_PinHeader_2.54mm:PinHeader_1x15_P2.54mm_Vertical, symbol controller_motion_pcb-rescue:Conn_01x15_Male-Connector
- removed P0, P1, P2, P3, P4, P5, P6, P7: Conn_01x03, Connector_JST:JST_EH_B3B-EH-A_1x03_P2.50mm_Vertical, symbol controller_motion_pcb-rescue:Conn_01x03-Connector_Generic
- removed mux1, mux2, mux3, mux4: 74HC4051, Package_DIP:DIP-16_W7.62mm, symbol controller_motion_pcb-rescue:74HC4051-74xx
- added C1, C5, C6, C7, C8, C9: 100nF, Capacitor_THT:C_Disc_D7.0mm_W2.5mm_P5.00mm, symbol Device:C
- added C2, C3: 22pF, Capacitor_THT:C_Disc_D7.0mm_W2.5mm_P5.00mm, symbol Device:C
- added C4: 10uH, Capacitor_THT:CP_Radial_D5.0mm_P2.00mm, symbol Device:CP
- added J1: ICSP INTERFACE, Connector_PinHeader_2.54mm:PinHeader_1x04_P2.54mm_Vertical, symbol Connector_Generic:Conn_01x04
- added J2: I2C INTERFACE MSTR, Connector_PinHeader_2.54mm:PinHeader_1x05_P2.54mm_Horizontal, symbol Connector_Generic:Conn_01x05
- added J3: I2C INTERFACE SLAV, Connector_PinSocket_2.54mm:PinSocket_1x05_P2.54mm_Horizontal, symbol Connector_Generic:Conn_01x05
- added J4: Conn_01x02_Male, Connector_PinHeader_2.54mm:PinHeader_1x02_P2.54mm_Horizontal, symbol Connector:Conn_01x02_Male
- added J5: Conn_01x02_Female, Connector_PinSocket_2.54mm:PinSocket_1x02_P2.54mm_Horizontal, symbol Connector:Conn_01x02_Female
- added J6: Conn_01x06_Female, Connector_JST:JST_PH_B5B-PH-K_1x05_P2.00mm_Vertical, symbol Connector:Conn_01x05_Female
- added L1: 10uH, Inductor_THT:L_Axial_L7.0mm_D3.3mm_P10.16mm_Horizontal_Fastron_MICC, symbol Device:L
- added R1: 0, Resistor_THT:R_Axial_DIN0207_L6.3mm_D2.5mm_P10.16mm_Horizontal, symbol Device:R
- added R10, R13, R16, R7: 165, Resistor_THT:R_Axial_DIN0207_L6.3mm_D2.5mm_P10.16mm_Horizontal, symbol Device:R
- added R11, R14, R17, R8: 155, Resistor_THT:R_Axial_DIN0207_L6.3mm_D2.5mm_P10.16mm_Horizontal, symbol Device:R
- added R12, R15, R18, R9: 100, Resistor_THT:R_Axial_DIN0207_L6.3mm_D2.5mm_P10.16mm_Horizontal, symbol Device:R
- added R19, R20: 27k, Resistor_THT:R_Axial_DIN0207_L6.3mm_D2.5mm_P10.16mm_Horizontal, symbol Device:R
- added R21, R3, R4, R5, R6: 4.7k, Resistor_THT:R_Axial_DIN0207_L6.3mm_D2.5mm_P10.16mm_Horizontal, symbol Device:R
- added R22, R23: 10k, Resistor_THT:R_Axial_DIN0207_L6.3mm_D2.5mm_P10.16mm_Horizontal, symbol Device:R
- added S1, S2, S3, S4: 228CMVARGBFR, flex-Ambisonic:228CMVARGBFR, symbol btn-matrix-rescue:228CMVARGBFR
- added SW1: Rotary_Encoder_Switch, MOUSERfootprintANDsymbol:PEC11R4230KS0024, symbol Device:Rotary_Encoder_Switch
- added U1: ATtiny861V-10SU, Package_SO:SOIC-20W_7.5x12.8mm_P1.27mm, symbol flex_AmbisonicLib:ATtiny861V-10SU
- added U2, U3: TPIC6C595-SOIC, Package_SO:SOIC-16_3.9x9.9mm_P1.27mm, symbol flex_AmbisonicLib:TPIC6C595-SOIC
- added Y1: Crystal, Crystal:Crystal_HC49-U_Vertical, symbol Device:Crystal
Connections:
- net GND: now also C1.1, C2.1, C3.1, C4.2, C5.1, C6.1, C7.2, C8.2, C9.2, J2.2 (Pin_2), J2.4 (Pin_4), J3.2 (Pin_2), J3.4 (Pin_4), J4.2 (Pin_2), J5.2 (Pin_2), J6.1 (Pin_1), J6.3 (Pin_3), S1.2 (COM_1), S2.1 (COM_1), S3.2 (COM_1), S4.1 (COM_1), SW1.C, SW1.S1, U1.16 (AGND), U1.6 (GND), U2.16 (GND), U3.16 (GND)
- new net: R3.2, S1.3 (COM_2)
- new net: R9.1, S1.5 (K_B)
- new net: R7.1, S1.6 (K_R)
- new net: R8.1, S1.8 (K_G)
- new net: R4.2, S2.3 (COM_2)
- new net: R12.1, S2.5 (K_B)
- new net: R10.1, S2.6 (K_R)
- new net: R11.1, S2.8 (K_G)
- new net: R5.2, S3.3 (COM_2)
- new net: R15.1, S3.5 (K_B)
- new net: R13.1, S3.6 (K_R)
- new net: R14.1, S3.8 (K_G)
- new net: R6.2, S4.4 (COM_2)
- new net: R18.1, S4.5 (K_B)
- new net: R16.1, S4.6 (K_R)
- new net: R17.1, S4.8 (K_G)
- new net: R19.2, SW1.A
- new net: R20.2, SW1.B
- new net: R21.1, SW1.S2
- new net: R23.1, U3.7 (~CLR~), U3.8 (~G~)
- new net: C5.2, L1.1, U1.15 (AVCC)
- new net: R11.2, U2.11 (DRAIN4)
- new net: R12.2, U2.14 (DRAIN7)
- new net: R13.2, U3.3 (DRAIN0)
- new net: R16.2, U3.6 (DRAIN3)
- new net: R14.2, U3.4 (DRAIN1)
- new net: R17.2, U3.11 (DRAIN4)
- new net: R15.2, U3.5 (DARIN2)
- new net: R18.2, U3.12 (DARIN5)
- new net: R22.1, U2.7 (~CLR~), U2.8 (~G~)
- new net: U2.9 (SEROUT), U3.2 (SERIN)
- new net ADC0: J6.4 (Pin_4), U1.11 (ADC6/PA7)
- new net ADC1: J6.2 (Pin_2), U1.12 (ADC5/PA6)
- new net ATM_VCC: C1.2, C4.1, C8.1, C9.1, J2.5 (Pin_5), J3.5 (Pin_5), J4.1 (Pin_1), J5.1 (Pin_1), J6.5 (Pin_5), L1.2, R22.2, R23.2, S1.7 (Anode), S2.7 (Anode), S3.7 (Anode), S4.7 (Anode), U1.5 (VCC), U2.1 (VCC), U3.1 (VCC)
- new net ENCA: C6.2, R19.1, U1.9 (PB6)
- new net ENCB: C7.1, R1.2, R20.1
- new net ENCSW: R21.2, U1.13 (ADC4/PA5)
- new net MISO: J1.2 (Pin_2), R3.1, U1.2 (MISO/PB1)
- new net MOSI: J1.3 (Pin_3), U1.1 (MOSI/PB0), U2.2 (SERIN)
- new net PB1: R4.1, U1.19 (ADC1/PA1)
- new net PB2: R5.1, U1.14 (ADC3/PA4)
- new net PB3: R6.1, U1.17 (AREF/PA3)
- new net PSHFCLK: J1.1 (Pin_1), U1.3 (SCL/SCK/PB2), U2.15 (SRCK), U3.15 (SRCK)
- new net PSHFUDATE: U1.4 (PB3), U2.10 (RCK), U3.10 (RCK)
- new net RESET: J1.4 (Pin_4), R1.1, U1.10 (~RESET~/PB7)
- new net S1_G: R8.2, U2.4 (DRAIN1)
- new net S1_R: R7.2, U2.5 (DARIN2)
- new net S1_b: R9.2, U2.3 (DRAIN0)
- new net S2_R: R10.2, U2.13 (DRAIN6)
- new net SCL: J2.3 (Pin_3), J3.3 (Pin_3), U1.18 (SCL/PA2)
- new net SDA: J2.1 (Pin_1), J3.1 (Pin_1), U1.20 (SDA/ADC0/PA0)
- new net XTAL1: C2.2, U1.7 (XTAL1/PB4), Y1.1
- new net XTAL2: C3.2, U1.8 (XTAL2/PB5), Y1.2
- no-connect marks 26 -> 12

Commit message: MCU and Controller board done
Parts:
- removed C1, C5: 100nF, Capacitor_THT:C_Disc_D7.0mm_W2.5mm_P5.00mm, symbol Device:C
- removed C2, C3: 22pF, Capacitor_THT:C_Disc_D7.0mm_W2.5mm_P5.00mm, symbol Device:C
- removed C4: 10uH, Capacitor_THT:CP_Radial_D5.0mm_P2.00mm, symbol Device:CP
- removed J1: ICSP INTERFACE, Connector_PinHeader_2.54mm:PinHeader_1x04_P2.54mm_Vertical, symbol Connector_Generic:Conn_01x04
- removed J2: I2C INTERFACE MSTR, Connector_PinHeader_2.54mm:PinHeader_1x05_P2.54mm_Horizontal, symbol Connector_Generic:Conn_01x05
- removed J3: I2C INTERFACE SLAV, Connector_PinSocket_2.54mm:PinSocket_1x05_P2.54mm_Horizontal, symbol Connector_Generic:Conn_01x05
- removed J4: Conn_01x02_Male, Connector_PinHeader_2.54mm:PinHeader_1x02_P2.54mm_Horizontal, symbol Connector:Conn_01x02_Male
- removed J5: Conn_01x02_Female, Connector_PinSocket_2.54mm:PinSocket_1x02_P2.54mm_Horizontal, symbol Connector:Conn_01x02_Female
- removed L1: 10uH, Inductor_THT:L_Axial_L7.0mm_D3.3mm_P10.16mm_Horizontal_Fastron_MICC, symbol Device:L
- removed R1: 0, Resistor_THT:R_Axial_DIN0207_L6.3mm_D2.5mm_P10.16mm_Horizontal, symbol Device:R
- removed R21, R3, R4, R5, R6: 4.7k, Resistor_THT:R_Axial_DIN0207_L6.3mm_D2.5mm_P10.16mm_Horizontal, symbol Device:R
- removed U1: ATtiny861V-10SU, Package_SO:SOIC-20W_7.5x12.8mm_P1.27mm, symbol flex_AmbisonicLib:ATtiny861V-10SU
- removed Y1: Crystal, Crystal:Crystal_HC49-U_Vertical, symbol Device:Crystal
- added J1, J2: Conn_01x09_Male, Connector_PinHeader_2.54mm:PinHeader_1x09_P2.54mm_Vertical, symbol Connector:Conn_01x09_Male
- C1: renamed from C6; footprint Capacitor_THT:C_Disc_D7.0mm_W2.5mm_P5.00mm -> Capacitor_SMD:C_1206_3216Metric_Pad1.33x1.80mm_HandSolder
- C2: renamed from C7; footprint Capacitor_THT:C_Disc_D7.0mm_W2.5mm_P5.00mm -> Capacitor_SMD:C_1206_3216Metric_Pad1.33x1.80mm_HandSolder
- C3: renamed from C8; footprint Capacitor_THT:C_Disc_D7.0mm_W2.5mm_P5.00mm -> Capacitor_SMD:C_1206_3216Metric_Pad1.33x1.80mm_HandSolder
- C4: renamed from C9; footprint Capacitor_THT:C_Disc_D7.0mm_W2.5mm_P5.00mm -> Capacitor_SMD:C_1206_3216Metric_Pad1.33x1.80mm_HandSolder
- R10: renamed from R12; footprint Resistor_THT:R_Axial_DIN0207_L6.3mm_D2.5mm_P10.16mm_Horizontal -> Resistor_SMD:R_1206_3216Metric_Pad1.30x1.75mm_HandSolder
- R11: renamed from R13; footprint Resistor_THT:R_Axial_DIN0207_L6.3mm_D2.5mm_P10.16mm_Horizontal -> Resistor_SMD:R_1206_3216Metric_Pad1.30x1.75mm_HandSolder
- R12: renamed from R14; footprint Resistor_THT:R_Axial_DIN0207_L6.3mm_D2.5mm_P10.16mm_Horizontal -> Resistor_SMD:R_1206_3216Metric_Pad1.30x1.75mm_HandSolder
- R13: renamed from R15; footprint Resistor_THT:R_Axial_DIN0207_L6.3mm_D2.5mm_P10.16mm_Horizontal -> Resistor_SMD:R_1206_3216Metric_Pad1.30x1.75mm_HandSolder
- R14: renamed from R16; footprint Resistor_THT:R_Axial_DIN0207_L6.3mm_D2.5mm_P10.16mm_Horizontal -> Resistor_SMD:R_1206_3216Metric_Pad1.30x1.75mm_HandSolder
- R15: renamed from R17; footprint Resistor_THT:R_Axial_DIN0207_L6.3mm_D2.5mm_P10.16mm_Horizontal -> Resistor_SMD:R_1206_3216Metric_Pad1.30x1.75mm_HandSolder
- R16: renamed from R18; footprint Resistor_THT:R_Axial_DIN0207_L6.3mm_D2.5mm_P10.16mm_Horizontal -> Resistor_SMD:R_1206_3216Metric_Pad1.30x1.75mm_HandSolder
- R17: renamed from R19; footprint Resistor_THT:R_Axial_DIN0207_L6.3mm_D2.5mm_P10.16mm_Horizontal -> Resistor_SMD:R_1206_3216Metric_Pad1.30x1.75mm_HandSolder
- R18: renamed from R20; footprint Resistor_THT:R_Axial_DIN0207_L6.3mm_D2.5mm_P10.16mm_Horizontal -> Resistor_SMD:R_1206_3216Metric_Pad1.30x1.75mm_HandSolder
- R20: renamed from R22; footprint Resistor_THT:R_Axial_DIN0207_L6.3mm_D2.5mm_P10.16mm_Horizontal -> Resistor_SMD:R_1206_3216Metric_Pad1.30x1.75mm_HandSolder
- R21: renamed from R23; footprint Resistor_THT:R_Axial_DIN0207_L6.3mm_D2.5mm_P10.16mm_Horizontal -> Resistor_SMD:R_1206_3216Metric_Pad1.30x1.75mm_HandSolder
- R5: renamed from R7; footprint Resistor_THT:R_Axial_DIN0207_L6.3mm_D2.5mm_P10.16mm_Horizontal -> Resistor_SMD:R_1206_3216Metric_Pad1.30x1.75mm_HandSolder
- R6: renamed from R8; footprint Resistor_THT:R_Axial_DIN0207_L6.3mm_D2.5mm_P10.16mm_Horizontal -> Resistor_SMD:R_1206_3216Metric_Pad1.30x1.75mm_HandSolder
- R7: renamed from R9; footprint Resistor_THT:R_Axial_DIN0207_L6.3mm_D2.5mm_P10.16mm_Horizontal -> Resistor_SMD:R_1206_3216Metric_Pad1.30x1.75mm_HandSolder
- R8: renamed from R10; footprint Resistor_THT:R_Axial_DIN0207_L6.3mm_D2.5mm_P10.16mm_Horizontal -> Resistor_SMD:R_1206_3216Metric_Pad1.30x1.75mm_HandSolder
- R9: renamed from R11; footprint Resistor_THT:R_Axial_DIN0207_L6.3mm_D2.5mm_P10.16mm_Horizontal -> Resistor_SMD:R_1206_3216Metric_Pad1.30x1.75mm_HandSolder
- S1, S2, S3, S4: footprint flex-Ambisonic:228CMVARGBFR -> MOUSERfootprintANDsymbol:228CMVARGBFR
- renumbered J6 to J3, U2 to U1, U3 to U2
Connections:
- net labels added: GND-power, S2_B, S2_G, S3_B, S3_G, S3_R, S4_B, S4_G, S4_R
- net labels removed: ATM_VCC, MISO, MOSI, RESET, SCK, SCL, SDA, XTAL1, XTAL2
- wire segments 83 -> 37
- no-connect marks 12 -> 13
Other:
- moved on the sheet: R11, R12, R13, R14, R15, R16, S3, S4

Commit message: first protoype
Changed lines of the file:
@@
 Text GLabel 2750 4550 0    50   Input ~ 0
 ADC0
-Text GLabel 2750 4750 0    50   Input ~ 0
+Text GLabel 2750 4350 0    50   Input ~ 0
 ADC1
 Text GLabel 2750 4150 0    50   Input ~ 0
@@
 Text GLabel 3650 4850 2    50   Input ~ 0
 PB3
-Text GLabel 2750 4350 0    50   Input ~ 0
+Text GLabel 2750 4650 0    50   Input ~ 0
 PB1
 Text GLabel 3650 4150 2    50   Input ~ 0
@@
 Text GLabel 3650 4650 2    50   Input ~ 0
 VCC
-Text GLabel 2750 4650 0    50   Input ~ 0
+Text GLabel 2750 4450 0    50   Input ~ 0
 GND
 Text GLabel 2750 4850 0    50   Input ~ 0
 GND
-Text GLabel 2750 4450 0    50   Input ~ 0
+Text GLabel 2750 4750 0    50   Input ~ 0
 VCC
 $Comp
