File: moc/Mainboard-pcb/controller_motion_pcb.kicad_pcb (KiCad board)
At the start: 2 copper layers, 30 x 156 mm, 44 parts, among them J1 SPI_Female, J2 SPI_Male, J3 Conn_01x06_Female, J4 UPDI_Interface, J5 Programm_Jumper, SW1 Rotary_Encoder_Switch, U1 TPIC6C595-SOIC, U2 TPIC6C595-SOIC, U3 ATtiny1626

Commit message: clean up
Parts:
- moved J2 150.9 mm to (156.6, 175.9), turned to 0 degrees
- moved J1 150.8 mm to (138.6, 175.9), turned to 0 degrees
- moved R17 149.7 mm to (131.7, 27.8), turned to 0 degrees
- moved C1 142.9 mm to (131.7, 31.3), turned to 180 degrees
- moved REF** 141.7 mm to (142.8, 171.7), turned to 90 degrees
- moved SW1 140.6 mm to (143.7, 30.8), turned to -90 degrees
- moved C2 134.1 mm to (131.7, 35.8), turned to 0 degrees
- moved R18 127.3 mm to (131.7, 39.3), turned to 0 degrees
- moved REF** 113.2 mm to (133.6, 155.9), turned to 90 degrees
- moved R15 111.9 mm to (142.3, 156.7), turned to 90 degrees
- moved S4 111.8 mm to (143.7, 156.8), turned to 0 degrees
- moved R14 111.7 mm to (145.1, 156.8), turned to 90 degrees
- moved J3 111.5 mm to (145.7, 45.3), turned to 180 degrees
- moved REF** 108.7 mm to (138.5, 154.6), turned to 90 degrees
- moved J4 108.4 mm to (133.1, 153.3), turned to 180 degrees
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