File: a3motion/a3motion_buttonmatrix_pcb_v0.1/a3motion_buttonmatrix_v01.kicad_pcb (KiCad board)
At the start: 2 copper layers, 130 x 130 mm, 102 parts, among them J2 Conn_02x12_Odd_Even, U0 WS2811, U1 WS2811, U10 WS2811, U11 WS2811, U12 WS2811, U13 WS2811, U14 WS2811, U15 WS2811, U2 WS2811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

Commit message: ohl-s ready
Other:
- board text added: "https://github.com/a3-audio/a3-hardware A³ Motion - Buttonmatrix v0.1 Licensed under CERN-OHL-S v2"
Changed lines of the file:
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@@
     (rev "v.0.1")
     (company "A3 Audio UG (haftungsbeschränkt)")
+    (comment 3 "ttps://github.com/a3-audio/a3-hardware")
+    (comment 4 "Licensed under CERN-OHL-S v2")
   )
   (layers
@@
   (gr_line (start 157.37978 154.05078) (end 27.42978 154.05078) (layer "Edge.Cuts") (width 0.05))
   (gr_line (start 157.37978 24.07578) (end 157.37978 154.05078) (layer "Edge.Cuts") (width 0.05))
+  (gr_text "https://github.com/a3-audio/a3-hardware\n\nA³ Motion - Buttonmatrix v0.1\nLicensed under CERN-OHL-S v2\n" (at 94.521377 32.644439 -90) (layer "F.SilkS")
+    (effects (font (size 2 2) (thickness 0.2)) (justify left))
+  )
   (segment (start 78.30478 36.92578) (end 78.30478 38.92578) (width 0.25) (layer "B.Cu") (net 1))
   (segment (start 76.67478 38.92578) (end 78.30478 38.92578) (width 0.25) (layer "B.Cu") (net 1))
