File: a3motion/a3motion_mainboard_pcb_v0.1/a3motion_mainboard_v01.kicad_pcb (KiCad board)
At the start: 4 copper layers, 113 x 54 mm, 24 parts, among them J1 Conn_01x14_Male, J3 Conn_01x15_Male, P0 Conn_01x03, P1 Conn_01x03, P2 Conn_01x03, P3 Conn_01x03, P4 Conn_01x03, P5 Conn_01x03, P6 Conn_01x03, P7 Conn_01x03

Commit message: ohl-s ready
Other:
- board text added: "https://github.com/a3-audio/a3-hardware A³ Motion - Mainboard v0.1 Licensed under CERN-OHL-S v2"
Changed lines of the file:
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@@
     (rev "v.0.1")
     (company "A3 Audio UG (haftungsbeschränkt)")
+    (comment 3 "https://github.com/a3-audio/a3-hardware")
+    (comment 4 "Licensed under CERN-OHL-S v2")
   )
   (layers
@@
     (effects (font (size 7 7) (thickness 0.6)) (justify mirror))
   )
+  (gr_text "https://github.com/a3-audio/a3-hardware\n\nA³ Motion - Mainboard v0.1\nLicensed under CERN-OHL-S v2\n" (at 80.345001 58.965001) (layer "F.SilkS")
+    (effects (font (size 1 1) (thickness 0.1)) (justify left))
+  )
   (segment (start 168.38 47.88) (end 169.76 46.5) (width 0.25) (layer "B.Cu") (net 1))
