File: a3motion/a3motion_mainboard_pcb_v0.1/a3motion_mainboard_v01.kicad_sch (KiCad schematic)
At the start: 20 parts

Commit message: ohl-s ready
Parts:
- BtnMx1: value (none) -> Conn_02x09_Counter_Clockwise; footprint (none) -> Connector_IDC:IDC-Header_2x10_P2.54mm_Vertical
- CTR1: value (none) -> Teensy4.1; footprint (none) -> teensy:Teensy41
- ENC0, ENC1, ENC2, ENC3: value (none) -> Conn_01x05; footprint (none) -> Connector_JST:JST_EH_B5B-EH-A_1x05_P2.50mm_Vertical
- J1: value (none) -> Conn_01x14_Male; footprint (none) -> Connector_PinHeader_2.54mm:PinHeader_1x14_P2.54mm_Vertical
- J3: value (none) -> Conn_01x15_Male; footprint (none) -> Connector_PinHeader_2.54mm:PinHeader_1x15_P2.54mm_Vertical
- P0, P1, P2, P3, P4, P5, P6, P7: value (none) -> Conn_01x03; footprint (none) -> Connector_JST:JST_EH_B3B-EH-A_1x03_P2.50mm_Vertical
- mux1, mux2, mux3, mux4: value (none) -> 74HC4051; footprint (none) -> Package_DIP:DIP-16_W7.62mm
