File: a3mix/a3mix_mainboard_v02/a3mix.kicad_sch (KiCad schematic)
At the start: 160 parts

Commit message: A³ Mix draft license ohl-s
Parts:
- 3.3V_In1, 3.3V_Test1, 3.3V_Test2: value (none) -> Conn_01x02; footprint (none) -> Connector_JST:JST_XH_B2B-XH-AM_1x02_P2.50mm_Vertical
- C1, C2, C7: value (none) -> 100 uF; footprint (none) -> Capacitor_THT:CP_Radial_D10.0mm_P2.50mm
- C10, C11, C12, C3, C4, C5, C6, C8, C9: value (none) -> 100 nF; footprint (none) -> Capacitor_THT:CP_Radial_D5.0mm_P2.50mm
- FX-BTNs1, MuxCh1, MuxCh2, MuxCh3, MuxCh4, MuxCh5, fxEncBtns1: value (none) -> 74HC4051; footprint (none) -> Package_DIP:DIP-16_W7.62mm
- MuxCh1_1, MuxCh1_10, MuxCh1_11, MuxCh1_12, MuxCh1_13, MuxCh1_14, MuxCh1_15, MuxCh1_16, MuxCh1_17, MuxCh1_18, MuxCh1_19, MuxCh1_2, MuxCh1_20, MuxCh1_21, MuxCh1_22, MuxCh1_23, MuxCh1_24, MuxCh1_25, MuxCh1_26, MuxCh1_27, MuxCh1_28, MuxCh1_29, MuxCh1_3, MuxCh1_30, MuxCh1_31, MuxCh1_32, MuxCh1_33, MuxCh1_34, MuxCh1_35, MuxCh1_36, MuxCh1_37, MuxCh1_38, MuxCh1_39, MuxCh1_4, MuxCh1_40, MuxCh1_5, MuxCh1_6, MuxCh1_7, MuxCh1_8, MuxCh1_9, NeoPixel1, spare(28)1, spare(29)1: value (none) -> Conn_01x03; footprint (none) -> Connector_JST:JST_XH_B3B-XH-A_1x03_P2.50mm_Vertical
- R1, R10, R11, R12, R13, R14, R15, R16, R17, R19, R2, R20, R21, R22, R23, R24, R25, R26, R27, R28, R29, R3, R34, R35, R36, R37, R38, R39, R4, R40, R41, R42, R43, R44, R45, R46, R47, R48, R49, R5, R50, R51, R52, R53, R54, R55, R56, R57, R58, R59, R6, R60, R61, R62, R63, R64, R65, R66, R67, R7, R8, R9: value (none) -> 100k; footprint (none) -> Resistor_THT:R_Axial_DIN0207_L6.3mm_D2.5mm_P10.16mm_Horizontal
- R18, R30, R31, R32, R33: value (none) -> 500; footprint (none) -> Resistor_THT:R_Axial_DIN0207_L6.3mm_D2.5mm_P10.16mm_Horizontal
- U5: value (none) -> Teensy4.1; footprint (none) -> teensy:Teensy41
- VU_Matrix1: value (none) -> MAX7219 led matrix vu; footprint (none) -> Connector_JST:JST_XH_B5B-XH-A_1x05_P2.50mm_Vertical
- display_1, display_2: value (none) -> Conn_01x04; footprint (none) -> Connector_JST:JST_XH_B4B-XH-A_1x04_P2.50mm_Vertical
- fx1_btn1, fx1_btn2, fx1_btn3, fx1_btn4, fx2_btn1, fx2_btn2, fx2_btn3, fx2_btn4, pfl_btn_1, pfl_btn_2, pfl_btn_3, pfl_btn_4, pfl_btn_master1, pfl_led_1, pfl_led_2, pfl_led_3, pfl_led_4, pfl_led_master1: value (none) -> Conn_01x02; footprint (none) -> Connector_JST:JST_XH_B2B-XH-A_1x02_P2.50mm_Vertical
- fx1_enc1, fx1_enc2, fx1_enc3, fx2_enc1, fx2_enc2, fx2_enc3: value (none) -> Conn_01x05; footprint (none) -> Connector_JST:JST_XH_B5B-XH-A_1x05_P2.50mm_Vertical
